File: hardware/_autosave-iot_crockpot.kicad_pcb (KiCad board)
At the start: 2 copper layers, 9 parts, among them K1 G5LE-1, K2 G5LE-1, Q1 2N7002, Q2 2N7002, U1 AMS1117-3.3, U2 MOUDLE-SEEEDUINO-XIAO-ESP32C3

Commit message: Started schematic part selection
added XIAO ESP32-C3
added HLK-PM01 120VAC to 5VDC power module
added relays
added thermal couple sensor
Parts:
- added U3: MAX31855KASA, Package_SO:SOIC-8_3.9x4.9mm_P1.27mm, F.Cu at (165.0, 110.6)
- moved U2 17.9 mm to (176.3, 84.1)
Connections:
- U2 pad 12: unconnected-(U2-3V3-Pad12) -> +3V3
- U2 pad 13: unconnected-(U2-GND-Pad13) -> GND
